Commit message: update

File: src/robot_description/urdf/chassis.xacro (robot description, xacro)
@@ -38,5 +38,5 @@
         <origin xyz="0.0 0.0 0.0" rpy="0.0 0.0 0.0"/>
         <geometry>
-          <box size="0.45 0.38 0.15"/>
+          <box size="0.45 0.30 0.10"/>
         </geometry>
       </collision>
